File: hardware/mc68k_sbc.kicad_sch (KiCad schematic)
At the start: 92 parts, among them J1 EXP, J10 JTAG_Conn, J2 DE9_Pins, J6 I2C_Conn, J7 USB_C_Receptacle_USB2.0_14P, J8 SPI_Conn, SW2 Reset, SW3 Power Switch, U1 MC68000P/MC68010P, U10 28C256, U11 CH340N, U13 XC9572XL-xxVQx64, U14 MCP100-450D, U2 68681, U3 28C256, U4 AS6C4008-55PCN, U5 FT231XS, U6 MAX232, U7 PCF8584, U8 AS6C4008-55PCN, U9 AMS1117-3.3, Y1 CXO_DIP14, Y2 CXO_DIP8

Commit message: added bootord autoboot for bootloader, updated schematics
Parts:
- removed C9: 0.1uF, Capacitor_THT:C_Disc_D3.0mm_W1.6mm_P2.50mm, symbol Device:C
- removed D2, D3: LED, LED_THT:LED_D3.0mm, symbol Device:LED
- removed J6: I2C_Conn, Connector_PinHeader_2.54mm:PinHeader_1x04_P2.54mm_Vertical, symbol Connector:Conn_01x04_Pin
- removed R5, R6: 220R, Resistor_THT:R_Axial_DIN0204_L3.6mm_D1.6mm_P1.90mm_Vertical, symbol Device:R
- removed U5: FT231XS, Package_SO:SSOP-20_3.9x8.7mm_P0.635mm, symbol Interface_USB:FT231XS
- added J6: I2C_Conn, Package_DIP:DIP-20_W7.62mm, symbol Connector_Generic:Conn_01x04
Connections:
- net GND: now also U11.3 (GND), J6.4 (Pin_4)
- net RX_USB: now also U11.7 (RXD)
- net TX_USB: now also U11.6 (TXD)
- net VCC: now also U11.5 (VCC), J6.1 (Pin_1)
- net ~{RTS}_USB: now also U11.4 (~{RTS}); no longer U2.29 (OP0)
- net at R7.1, U7.2 (SDA): now also J6.2 (Pin_2)
- net at R8.2, U7.3 (SCL): now also J6.3 (Pin_3)
- net at R3.1: now also U11.2 (UD-)
- net at R4.1: now also U11.1 (UD+)
- net ~{CTS}_USB: no longer names the net of U2.7 (IP0)
Other:
- moved on the sheet: C10, C11, C12, C13, C14, C15, C16, C17, C18, C19, C20, C21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
